Commit message: Add a disk shaped link below magnet to prevent strange behaviour

File: mmuav_description/urdf/uav.gazebo.xacro (robot description, xacro)
@@ -58,9 +58,32 @@
   </gazebo>
   <xacro:if value="${mount_magnet}">
+    <joint name="electromagnet_joint" type="fixed">
+      <axis xyz="0 1 0" />
+      <origin xyz="0.0 0.0 -0.15" rpy="0 0 0"/>
+      <parent link="base_link"/>
+      <child link="electromagnet_actuator"/>
+    </joint>
+    <link name="electromagnet_actuator">
+      <inertial>
+      <origin xyz="0 0 0" rpy="0 0 0" />
+      <mass value="0.025"/>
+      <inertia ixx="0.0001" ixy="0" ixz="0" iyy ="0.0001" iyz = "0" izz = "0.0001" />
+      </inertial>
+      <collision name="collision">
+      <geometry>
+        <cylinder radius="0.08" length="0.035"/>
+      </geometry>
+      </collision>
+      <visual>
+      <geometry>
+        <cylinder radius="0.08" length="0.035"/>
+      </geometry>
+      </visual>
+    </link>
     <gazebo>
       <plugin name="dipole_magnet" filename="libstorm_gazebo_dipole_magnet.so">
-        <robotNamespace>uav</robotNamespace>
+        <robotNamespace>$(arg name)</robotNamespace>
         <bodyName>base_link</bodyName>
-        <dipole_moment>0 0 970</dipole_moment>
+        <dipole_moment>0 0 50</dipole_moment>
         <!-- Set to false if not using ROS -->
         <shouldPublish>true</shouldPublish>
